Commit message: 1.1

File: src/fang/urdf/base.urdf.xacro (robot description, xacro)
@@ -1,4 +1,4 @@
 <?xml version="1.0"?>
-<robot xmlns:xacro="http://www.ros.org/wiki/xacro">
+<robot xmlns:xacro="http://ros.org/wiki/xacro">
     <xacro:include filename="yuan.urdf.xacro"/>
     <xacro:macro name="base_xacro" params="length radius">
@@ -9,5 +9,5 @@
             <xacro:cylinder_inertia m="1.0" r="${radius}" h="${length}"/>
         </link>
-        <joint name="joint_name" type="fixed">
+        <joint name="joint_first" type="fixed">
             <origin xyz="0.0 0.0 ${length/2.0}" rpy="0.0 0.0 0.0"/>
             <parent link="base_footprint"/>

File: src/fang/urdf/car.urdf.xacro (robot description, xacro)
@@ -1,5 +1,9 @@
 <?xml version="1.0"?>
-<robot name="car" xmlns:xacro="http://ros.org/wiki/xacro">
+<robot xmlns:xacro="http://ros.org/wiki/xacro" name="car">
     <xacro:include filename="base.urdf.xacro"/>
+    <xacro:include filename="wheel/wheel.urdf.xacro"/>
     <xacro:base_xacro length="0.3" radius="0.3"/>
+    <xacro:wheel wheel_name="wheel_1" xyz="0.3 0.0 -0.15" axis_xyz="1.0 0.0 0.0" rpy="0.0 1.57079 0.0"/>
+    <xacro:wheel wheel_name="wheel_2" xyz="-0.15 0.25980 -0.15" axis_xyz="0.5 -0.86603 0.0" rpy="0.0 1.57079 2.09440"/>
+    <xacro:wheel wheel_name="wheel_3" xyz="-0.15 -0.25980 -0.15" axis_xyz="0.5 0.86603 0.0" rpy="0.0 1.57079 1.04720"/>
 </robot>

File: src/fang/urdf/yuan.urdf.xacro (robot description, xacro)
@@ -3,7 +3,7 @@
     <!-- 视觉 -->
     <!-- 方形 -->
-    <xacro:macro name="box_visual" params="x y z">
+    <xacro:macro name="box_visual" params="x y z rpy:='0 0.0 0.0'">
         <visual>
-            <origin xyz="0.0 0.0 0.0" rpy="0.0 0.0 0.0"/>
+            <origin xyz="0.0 0.0 0.0" rpy="${rpy}"/>
             <geometry>
                 <box size="${x} ${y} ${z}"/>
@@ -15,19 +15,19 @@
     </xacro:macro>
     <!-- 圆柱 -->
-    <xacro:macro name="cylinder_visual" params="r h">
+    <xacro:macro name="cylinder_visual" params="r h rpy:='0.0 0.0 0.0'">
         <visual>
-            <origin xyz="0.0 0.0 0.0" rpy="0.0 0.0 0.0"/>
+            <origin xyz="0.0 0.0 0.0" rpy="${rpy}"/>
             <geometry>
                 <cylinder radius="${r}" length="${h}"/>
             </geometry>
-            <material name="blue">
-                <color rgba="0.0 0.0 1.0 1.0"/>
+            <material name="white">
+                <color rgba="1.0 1.0 1.0 0.5"/>
             </material>
         </visual>
     </xacro:macro>
     <!-- 球 -->
-    <xacro:macro name="sphere_visual" params="r">
+    <xacro:macro name="sphere_visual" params="r rpy:='0.0 0.0 0.0'">
         <visual>
-            <origin xyz="0.0 0.0 0.0" rpy="0.0 0.0 0.0"/>
+            <origin xyz="0.0 0.0 0.0" rpy="${rpy}"/>
             <geometry>
                 <sphere radius="${r}"/>
@@ -40,7 +40,7 @@
     <!-- 碰撞 -->
     <!-- 方形 -->
-    <xacro:macro name="box_collision" params="x y z">
+    <xacro:macro name="box_collision" params="x y z rpy:='0.0 0.0 0.0'">
         <collision>
-            <origin xyz="0.0 0.0 0.0" rpy="0.0 0.0 0.0"/>
+            <origin xyz="0.0 0.0 0.0" rpy="${rpy}"/>
             <geometry>
                 <box size="${x} ${y} ${z}"/>
@@ -49,7 +49,7 @@
     </xacro:macro>
     <!-- 圆柱 -->
-    <xacro:macro name="cylinder_collision" params="r h">
+    <xacro:macro name="cylinder_collision" params="r h rpy:='0.0 0.0 0.0'">
         <collision>
-            <origin xyz="0.0 0.0 0.0" rpy="0.0 0.0 0.0"/>
+            <origin xyz="0.0 0.0 0.0" rpy="${rpy}"/>
             <geometry>
                 <cylinder radius="${r}" length="${h}"/>
@@ -58,7 +58,7 @@
     </xacro:macro>
     <!-- 球 -->
-    <xacro:macro name="sphere_collision" params="r">
+    <xacro:macro name="sphere_collision" params="r rpy:='0.0 0.0 0.0'">
         <collision>
-            <origin xyz="0.0 0.0 0.0" rpy="0.0 0.0 0.0"/>
+            <origin xyz="0.0 0.0 0.0" rpy="${rpy}"/>
             <geometry>
                 <sphere radius="${r}"/>
@@ -68,7 +68,7 @@
     <!-- 惯性 -->
     <!-- 方形 -->
-    <xacro:macro name="box_inertia" params="m x y z">
+    <xacro:macro name="box_inertia" params="m x y z rpy:='0.0 0.0 0.0'">
         <inertial>
-            <origin xyz="0.0 0.0 0.0" rpy="0.0 0.0 0.0"/>
+            <origin xyz="0.0 0.0 0.0" rpy="${rpy}"/>
             <mass value="${m}" />
             <inertia ixx="${(m/12) * (y*y + z*z)}" ixy="0.0" ixz="0.0" iyy="${(m/12) * (x*x + z*z)}" iyz="0.0" izz="${(m/12) * (x*x + y*y)}" />
@@ -76,7 +76,7 @@
     </xacro:macro>
     <!-- 圆柱 -->
-    <xacro:macro name="cylinder_inertia" params="m r h">
+    <xacro:macro name="cylinder_inertia" params="m r h rpy:='0.0 0.0 0.0'">
         <inertial>
-            <origin xyz="0.0 0.0 0.0" rpy="0.0 0.0 0.0"/>
+            <origin xyz="0.0 0.0 0.0" rpy="${rpy}"/>
             <mass value="${m}" />
             <inertia ixx="${(m/12) * (3*r*r + h*h)}" ixy="0" ixz="0" iyy="${(m/12) * (3*r*r + h*h)}" iyz="0" izz="${(m/2) * (r*r)}" />
@@ -84,7 +84,7 @@
     </xacro:macro>
     <!-- 球 -->
-    <xacro:macro name="sphere_inertia" params="m r">
+    <xacro:macro name="sphere_inertia" params="m r rpy:='0.0 0.0 0.0'">
         <inertial>
-            <origin xyz="0.0 0.0 0.0" rpy="0.0 0.0 0.0"/>
+            <origin xyz="0.0 0.0 0.0" rpy="${rpy}"/>
             <mass value="${m}" />
             <inertia ixx="${(2/5) * m * (r*r)}" ixy="0.0" ixz="0.0" iyy="${(2/5) * m * (r*r)}" iyz="0.0" izz="${(2/5) * m * (r*r)}" />

Commit message: 1.3

File: src/fang/urdf/base.urdf.xacro (robot description, xacro)
@@ -6,9 +6,9 @@
         <link name="base_link">
             <xacro:cylinder_visual r="${radius}" h="${length}"/>
-            <xacro:cylinder_collision r="${radius}" h="${length}"/>
-            <xacro:cylinder_inertia m="1.0" r="${radius}" h="${length}"/>
+            <xacro:cylinder_collision r="${radius/2}" h="${length}"/>
+            <xacro:cylinder_inertia m="1.0" r="${radius/2}" h="${length}"/>
         </link>
         <joint name="joint_first" type="fixed">
-            <origin xyz="0.0 0.0 ${length/2.0}" rpy="0.0 0.0 0.0"/>
+            <origin xyz="0.0 0.0 0.075" rpy="0.0 0.0 0.0"/>
             <parent link="base_footprint"/>
             <child link="base_link"/>

File: src/fang/urdf/car.urdf.xacro (robot description, xacro)
@@ -3,7 +3,7 @@
     <xacro:include filename="base.urdf.xacro"/>
     <xacro:include filename="wheel/wheel.urdf.xacro"/>
-    <xacro:base_xacro length="0.3" radius="0.3"/>
-    <xacro:wheel wheel_name="wheel_1" xyz="0.3 0.0 -0.15" axis_xyz="1.0 0.0 0.0" rpy="0.0 1.57079 0.0"/>
-    <xacro:wheel wheel_name="wheel_2" xyz="-0.15 0.25980 -0.15" axis_xyz="0.5 -0.86603 0.0" rpy="0.0 1.57079 2.09440"/>
-    <xacro:wheel wheel_name="wheel_3" xyz="-0.15 -0.25980 -0.15" axis_xyz="0.5 0.86603 0.0" rpy="0.0 1.57079 1.04720"/>
+    <xacro:base_xacro length="0.05" radius="0.185"/>
+    <xacro:wheel wheel_name="wheel_1" xyz="0.185 0.0 0" axis_xyz="1.0 0.0 0.0" rpy="0.0 1.57079 0.0"/>
+    <xacro:wheel wheel_name="wheel_2" xyz="-0.0925 0.16021 0.0" axis_xyz="0.5 -0.86603 0.0" rpy="0.0 1.57079 2.09440"/>
+    <xacro:wheel wheel_name="wheel_3" xyz="-0.0925 -0.16021 0.0" axis_xyz="0.5 0.86603 0.0" rpy="0.0 1.57079 1.04720"/>
 </robot>

File: src/fang/urdf/wheel/wheel.urdf.xacro (robot description, xacro)
@@ -4,6 +4,6 @@
     <xacro:macro name="wheel" params="wheel_name xyz axis_xyz rpy:='0 0.0 0.0'">
         <link name="${wheel_name}_link">
-            <xacro:cylinder_visual r="0.1" h="0.03" rpy="${rpy}"/>
-            <xacro:cylinder_collision r="0.1" h="0.03" rpy="${rpy}"/>
+            <xacro:cylinder_visual r="0.075" h="0.04" rpy="${rpy}"/>
+            <xacro:cylinder_collision r="0.075" h="0.04" rpy="${rpy}"/>
         </link>
         <joint name="${wheel_name}_joint" type="continuous">
